Commit message: minor changes for compilation

File: msl_rotors_description/urdf/firefly_and_ball.xacro (robot description, xacro)
@@ -21,5 +21,5 @@
   <xacro:property name="rotor_velocity_slowdown_sim" value="10" />
   <xacro:property name="use_mesh_file" value="true" />
-  <xacro:property name="mesh_file" value="package://ec_rotors_description/meshes/firefly_and_ball.dae" />
+  <xacro:property name="mesh_file" value="package://msl_rotors_description/meshes/firefly_and_ball.dae" />
   <xacro:property name="mass" value="1.5" /> <!-- [kg] -->
   <xacro:property name="body_width" value="0.1" /> <!-- [m] -->
